Commit message: Da fix xong loi dieu khien bi lat ngua

File: description/cauhinh_robot.xacro (robot description, xacro)
@@ -5,5 +5,5 @@
     <xacro:property name="rong" value="0.23"/>
     <xacro:property name="cao" value="0.15"/>
-    <xacro:property name="KhoiLuongKhung" value="1.0"/>
+    <xacro:property name="KhoiLuongKhung" value="2.0"/>
     <xacro:property name="do_rong_banh_xe" value="0.027"/>
     <xacro:property name="ban_kinh_banh_xe" value="0.0325"/>
@@ -22,6 +22,5 @@
         <origin xyz="0 0 0" rpy="0 0 0"/>
     </joint>
-    <link name="base_footprint">
-    </link>
+    <link name="base_footprint"></link>
     <joint name="khung_joint" type="fixed">
         <parent link="base_link"/>
@@ -43,7 +42,8 @@
             </geometry>
         </collision>
-            <xacro:quan_tinh_hinh_hop mass="${KhoiLuongKhung}" x="${dai}" y="${rong}" z="${cao}">
-            <origin xyz="${dai/2} 0 ${cao/2}" rpy="0 0 0"/>
-        </xacro:quan_tinh_hinh_hop>
+        <xacro:quan_tinh_hinh_hop mass="${KhoiLuongKhung}" x="${dai}" y="${rong}" z="${cao}">
+        <!-- <origin xyz="${dai/2} 0 0.0" rpy="0 0 0"/> -->
+        <origin xyz="${dai/2} 0 ${ban_kinh_banh_xe}" rpy="0 0 0"/>
+    </xacro:quan_tinh_hinh_hop>
     </link>
     <gazebo reference="khung">
@@ -55,4 +55,5 @@
         <origin xyz="0 ${rong/2} 0" rpy="-${pi/2} 0 0" />
         <axis xyz="0 0 1"/>
+        <dynamics damping="0.1" friction="0.1"/>
     </joint>
     <link name="Banh_trai">
@@ -80,4 +81,5 @@
         <origin xyz="0 -${rong/2} 0" rpy="${pi/2} 0 0" />
         <axis xyz="0 0 -1"/>
+        <dynamics damping="0.1" friction="0.1"/>
     </joint>
     <link name="Banh_phai">
@@ -116,5 +118,4 @@
                 <sphere radius="${BK_BDH}"/>
             </geometry>
-            <material name="black"/>
         </collision>
         <xacro:quan_tinh_hinh_cau mass="${KL_BDH}" radius="${BK_BDH}">
@@ -124,6 +125,6 @@
     <gazebo reference="BDH_trc">
         <material>Gazebo/Black</material>
-        <mu1 value="0.001"/>
-        <mu2 value="0.001"/>
+        <mu1>0.0</mu1>
+        <mu2>0.0</mu2>
     </gazebo>
     <joint name="BDH_sau_joint" type="fixed">
@@ -143,5 +144,4 @@
                 <sphere radius="${BK_BDH}"/>
             </geometry>
-            <material name="black"/>
         </collision>
         <xacro:quan_tinh_hinh_cau mass="${KL_BDH}" radius="${BK_BDH}">
@@ -151,6 +151,6 @@
     <gazebo reference="BDH_sau">
         <material>Gazebo/Black</material>
-        <mu1 value="0.001"/>
-        <mu2 value="0.001"/>
+        <mu1>0.0</mu1>
+        <mu2>0.0</mu2>
     </gazebo>
 </robot>

Commit message: TAMJ  OK

File: description/cauhinh_robot.xacro (robot description, xacro)
@@ -44,5 +44,6 @@
         <xacro:quan_tinh_hinh_hop mass="${KhoiLuongKhung}" x="${dai}" y="${rong}" z="${cao}">
         <!-- <origin xyz="${dai/2} 0 0.0" rpy="0 0 0"/> -->
-        <origin xyz="${dai/2} 0 ${ban_kinh_banh_xe}" rpy="0 0 0"/>
+        <!-- <origin xyz="${dai/2} 0 ${ban_kinh_banh_xe}" rpy="0 0 0"/> -->
+        <origin xyz="${dai/2} 0 -0.05" rpy="0 0 0"/>
     </xacro:quan_tinh_hinh_hop>
     </link>
