Commit message: CHACS LAF OK ROI

File: description/lidar.xacro (robot description, xacro)
@@ -4,5 +4,5 @@
         <parent link="base_link"/>
         <child link="laser_frame"/>
-        <origin xyz="0.07 0 0.15" rpy="0 0 0"/>
+        <origin xyz="0.07 0 0.15" rpy="0 0 ${pi}"/>
     </joint>
     <link name="laser_frame">
